Commit message: add changes

File: src/robot_description/urdf/body.urdf.xacro (robot description, xacro)
@@ -1,10 +1,27 @@
 <robot name="body" xmlns:xacro="http://ros.org/wiki/xacro">
 <link name="base_link" />
+<!-- 質量、幅、高さ、奥行きを定義 -->
+<xacro:property name="b_m" value="1.68"/>
+<xacro:property name="b_w" value="0.07"/>
+<xacro:property name="b_h" value="0.13"/>
+<xacro:property name="b_d" value="0.055"/>
 <link name="body">
     <visual>
         <geometry>
-            <box size="0.07 0.13 0.055"/>
+            <box size="${b_w} ${b_h} ${b_d}"/>
         </geometry>
     </visual>
+    <collision>
+        <geometry>
+            <box size="${b_w} ${b_h} ${b_d}"/>
+        </geometry>
+    </collision>
+    <inertial>
+        <origin xyz="0.0 0.0 0.0" rpy="0.0 0.0 0.0"/>
+        <mass value="${b_m}"/>
+        <inertia ixx="${b_m*(b_h*b_h+b_d*b_d)/12}" ixy="0.0" ixz="0.0"
+                iyx="0.0" iyy="${b_m*(b_w*b_w+b_d*b_d)/12}" iyz="0.0"
+                izx="0.0" izy="0.0" izz="${b_m*(b_w*b_w+b_h*b_h)/12}"/>
+    </inertial>
 </link>
 <joint name="body_joint" type="fixed">

File: src/robot_description/urdf/wheel.urdf.xacro (robot description, xacro)
@@ -4,4 +4,5 @@
     <xacro:property name = "wheel_radius" value = "0.024" />
     <xacro:property name = "wheel_height" value = "0.008" />
+    <xacro:property name = "wheel_mass" value = "0.112" />
     <xacro:macro name = "wheel" params = "rl parent">
     <link name = "wheel_${rl}">
@@ -13,4 +14,18 @@
             </geometry>
         </visual>
+        <collision>
+            <geometry>
+                <cylinder
+                length = "${wheel_height}"
+                radius = "${wheel_radius}" />
+            </geometry>
+        </collision>
+        <inertial>
+            <origin xyz="0.0 0.0 0.0" rpy="0.0 0.0 0.0"/>
+            <mass value="${wheel_mass}"/>
+            <inertia ixx="${wheel_mass * (3 * wheel_radius * wheel_radius + wheel_height * wheel_height)/12}" ixy="0.0" ixz="0.0"
+                    iyx="0.0" iyy="${wheel_mass * (3 * wheel_radius * wheel_radius + wheel_height * wheel_height)/12}" iyz="0.0"
+                    izx="0.0" izy="0.0" izz="${wheel_mass * (wheel_radius * wheel_radius)/2}"/>
+        </inertial>
     </link>
     <joint name = "wheel_${rl}_joint" type = "continuous">
